Commit message: feat: expand simulation to full upper body including torso, head, and both arms

File: urdf/upper_body.urdf.xacro (robot description, xacro)
@@ -1,36 +1,71 @@
 <?xml version="1.0"?>
-<robot name="humanoid_arm" xmlns:xacro="http://ros.org/wiki/xacro">
+<robot name="humanoid_upper_body" xmlns:xacro="http://ros.org/wiki/xacro">
   <xacro:include filename="$(find dexhandv2_description)/urdf/dexhandv2_right.xacro"/>
   <link name="world"/>
-  <!-- Torso / Shoulder Base -->
-  <joint name="shoulder_yaw" type="revolute">
+  <!-- Pelvis (Base of the upper body) -->
+  <joint name="pelvis_joint" type="fixed">
     <parent link="world"/>
-    <child link="shoulder_link"/>
-    <origin xyz="0 0 0.5" rpy="0 0 0"/>
+    <child link="pelvis"/>
+    <origin xyz="0 0 1.0" rpy="0 0 0"/>
+  </joint>
+  <link name="pelvis">
+    <visual>
+      <geometry>
+        <box size="0.2 0.3 0.1"/>
+      </geometry>
+      <material name="blue">
+        <color rgba="0.2 0.2 0.8 1.0"/>
+      </material>
+    </visual>
+  </link>
+  <!-- Torso (Stomach to Chest) -->
+  <joint name="waist_yaw" type="revolute">
+    <parent link="pelvis"/>
+    <child link="torso"/>
+    <origin xyz="0 0 0.05" rpy="0 0 0"/>
     <axis xyz="0 0 1"/>
     <limit lower="-1.57" upper="1.57" effort="10" velocity="3"/>
   </joint>
-  <link name="shoulder_link">
+  <link name="torso">
+    <visual>
+      <origin xyz="0 0 0.2" rpy="0 0 0"/>
+      <geometry>
+        <box size="0.15 0.3 0.4"/>
+      </geometry>
+      <material name="blue"/>
+    </visual>
+  </link>
+  <!-- Neck & Head -->
+  <joint name="neck_pitch" type="revolute">
+    <parent link="torso"/>
+    <child link="head"/>
+    <origin xyz="0 0 0.45" rpy="0 0 0"/>
+    <axis xyz="0 1 0"/>
+    <limit lower="-0.78" upper="0.78" effort="10" velocity="3"/>
+  </joint>
+  <link name="head">
+    <visual>
+      <origin xyz="0 0 0.1" rpy="0 0 0"/>
+      <geometry>
+        <sphere radius="0.1"/>
+      </geometry>
+      <material name="skin">
+        <color rgba="0.9 0.7 0.6 1.0"/>
+      </material>
+    </visual>
+  </link>
+  <!-- Right Arm -->
+  <!-- Right Shoulder Base -->
+  <joint name="r_shoulder_yaw" type="revolute">
+    <parent link="torso"/>
+    <child link="r_shoulder_link"/>
+    <origin xyz="0 -0.2 0.35" rpy="0 0 0"/>
+    <axis xyz="0 0 1"/>
+    <limit lower="-1.57" upper="1.57" effort="10" velocity="3"/>
+  </joint>
+  <link name="r_shoulder_link">
     <visual>
       <geometry>
         <sphere radius="0.06"/>
-      </geometry>
-      <material name="white">
-        <color rgba="0.9 0.9 0.9 1.0"/>
-      </material>
-    </visual>
-  </link>
-  <joint name="shoulder_pitch" type="revolute">
-    <parent link="shoulder_link"/>
-    <child link="bicep"/>
-    <origin xyz="0 0 0" rpy="0 0 0"/>
-    <axis xyz="0 1 0"/>
-    <limit lower="-3.14" upper="3.14" effort="10" velocity="3"/>
-  </joint>
-  <link name="bicep">
-    <visual>
-      <origin xyz="0 0 -0.15" rpy="0 0 0"/>
-      <geometry>
-        <cylinder radius="0.04" length="0.3"/>
       </geometry>
       <material name="grey">
@@ -39,12 +74,28 @@
     </visual>
   </link>
-  <joint name="elbow_pitch" type="revolute">
-    <parent link="bicep"/>
-    <child link="forearm"/>
+  <joint name="r_shoulder_pitch" type="revolute">
+    <parent link="r_shoulder_link"/>
+    <child link="r_bicep"/>
+    <origin xyz="0 0 0" rpy="0 0 0"/>
+    <axis xyz="0 1 0"/>
+    <limit lower="-3.14" upper="3.14" effort="10" velocity="3"/>
+  </joint>
+  <link name="r_bicep">
+    <visual>
+      <origin xyz="0 0 -0.15" rpy="0 0 0"/>
+      <geometry>
+        <cylinder radius="0.04" length="0.3"/>
+      </geometry>
+      <material name="grey"/>
+    </visual>
+  </link>
+  <joint name="r_elbow_pitch" type="revolute">
+    <parent link="r_bicep"/>
+    <child link="r_forearm"/>
     <origin xyz="0 0 -0.3" rpy="0 0 0"/>
     <axis xyz="0 1 0"/>
     <limit lower="0" upper="2.5" effort="10" velocity="3"/>
   </joint>
-  <link name="forearm">
+  <link name="r_forearm">
     <visual>
       <origin xyz="0 0 -0.15" rpy="0 0 0"/>
@@ -55,7 +106,7 @@
     </visual>
   </link>
-  <!-- Connects to the DexHand's base_link -->
-  <joint name="wrist_roll" type="revolute">
-    <parent link="forearm"/>
+  <!-- Right Wrist Connects to DexHand's base_link -->
+  <joint name="r_wrist_roll" type="revolute">
+    <parent link="r_forearm"/>
     <child link="base_link"/>
     <origin xyz="0 0 -0.3" rpy="1.5708 0 0"/> <!-- Rotate so hand faces forward -->
@@ -63,3 +114,68 @@
     <limit lower="-1.57" upper="1.57" effort="10" velocity="3"/>
   </joint>
+  <!-- Left Arm -->
+  <!-- Left Shoulder Base -->
+  <joint name="l_shoulder_yaw" type="revolute">
+    <parent link="torso"/>
+    <child link="l_shoulder_link"/>
+    <origin xyz="0 0.2 0.35" rpy="0 0 0"/>
+    <axis xyz="0 0 1"/>
+    <limit lower="-1.57" upper="1.57" effort="10" velocity="3"/>
+  </joint>
+  <link name="l_shoulder_link">
+    <visual>
+      <geometry>
+        <sphere radius="0.06"/>
+      </geometry>
+      <material name="grey"/>
+    </visual>
+  </link>
+  <joint name="l_shoulder_pitch" type="revolute">
+    <parent link="l_shoulder_link"/>
+    <child link="l_bicep"/>
+    <origin xyz="0 0 0" rpy="0 0 0"/>
+    <axis xyz="0 1 0"/>
+    <limit lower="-3.14" upper="3.14" effort="10" velocity="3"/>
+  </joint>
+  <link name="l_bicep">
+    <visual>
+      <origin xyz="0 0 -0.15" rpy="0 0 0"/>
+      <geometry>
+        <cylinder radius="0.04" length="0.3"/>
+      </geometry>
+      <material name="grey"/>
+    </visual>
+  </link>
+  <joint name="l_elbow_pitch" type="revolute">
+    <parent link="l_bicep"/>
+    <child link="l_forearm"/>
+    <origin xyz="0 0 -0.3" rpy="0 0 0"/>
+    <axis xyz="0 1 0"/>
+    <limit lower="0" upper="2.5" effort="10" velocity="3"/>
+  </joint>
+  <link name="l_forearm">
+    <visual>
+      <origin xyz="0 0 -0.15" rpy="0 0 0"/>
+      <geometry>
+        <cylinder radius="0.035" length="0.3"/>
+      </geometry>
+      <material name="grey"/>
+    </visual>
+  </link>
+  <joint name="l_wrist_roll" type="revolute">
+    <parent link="l_forearm"/>
+    <child link="l_dummy_hand"/>
+    <origin xyz="0 0 -0.3" rpy="1.5708 0 0"/>
+    <axis xyz="0 0 1"/>
+    <limit lower="-1.57" upper="1.57" effort="10" velocity="3"/>
+  </joint>
+  <link name="l_dummy_hand">
+    <visual>
+      <geometry>
+        <box size="0.05 0.1 0.15"/>
+      </geometry>
+      <material name="grey"/>
+      <origin xyz="0 0.05 0" rpy="0 0 0"/>
+    </visual>
+  </link>
 </robot>

Commit message: fix: resolve jitter and implement 3-dof head rotation and jaw tracking

File: urdf/upper_body.urdf.xacro (robot description, xacro)
@@ -36,10 +36,26 @@
     </visual>
   </link>
-  <!-- Neck & Head -->
+  <!-- Neck & Head (3-DOF) -->
+  <joint name="neck_yaw" type="revolute">
+    <parent link="torso"/>
+    <child link="neck_link_1"/>
+    <origin xyz="0 0 0.45" rpy="0 0 0"/>
+    <axis xyz="0 0 1"/>
+    <limit lower="-1.57" upper="1.57" effort="10" velocity="3"/>
+  </joint>
+  <link name="neck_link_1"/>
   <joint name="neck_pitch" type="revolute">
-    <parent link="torso"/>
+    <parent link="neck_link_1"/>
+    <child link="neck_link_2"/>
+    <origin xyz="0 0 0" rpy="0 0 0"/>
+    <axis xyz="0 1 0"/>
+    <limit lower="-0.78" upper="0.78" effort="10" velocity="3"/>
+  </joint>
+  <link name="neck_link_2"/>
+  <joint name="neck_roll" type="revolute">
+    <parent link="neck_link_2"/>
     <child link="head"/>
-    <origin xyz="0 0 0.45" rpy="0 0 0"/>
-    <axis xyz="0 1 0"/>
+    <origin xyz="0 0 0" rpy="0 0 0"/>
+    <axis xyz="1 0 0"/>
     <limit lower="-0.78" upper="0.78" effort="10" velocity="3"/>
   </joint>
@@ -53,4 +69,21 @@
         <color rgba="0.9 0.7 0.6 1.0"/>
       </material>
+    </visual>
+  </link>
+  <!-- Jaw -->
+  <joint name="jaw_pitch" type="revolute">
+    <parent link="head"/>
+    <child link="jaw"/>
+    <origin xyz="0 0.05 0.05" rpy="0 0 0"/>
+    <axis xyz="1 0 0"/>
+    <limit lower="-0.5" upper="0.0" effort="10" velocity="3"/>
+  </joint>
+  <link name="jaw">
+    <visual>
+      <origin xyz="0 0.05 -0.05" rpy="0 0 0"/>
+      <geometry>
+        <box size="0.08 0.08 0.02"/>
+      </geometry>
+      <material name="skin"/>
     </visual>
   </link>

Commit message: feat: implement highly detailed realistic head with blinking, eyes, lips, and nose

File: urdf/upper_body.urdf.xacro (robot description, xacro)
@@ -60,4 +60,5 @@
     <limit lower="-0.78" upper="0.78" effort="10" velocity="3"/>
   </joint>
+  <!-- Head Base -->
   <link name="head">
     <visual>
@@ -71,19 +72,195 @@
     </visual>
   </link>
-  <!-- Jaw -->
+  <!-- Nose -->
+  <joint name="nose_fixed" type="fixed">
+    <parent link="head"/>
+    <child link="nose"/>
+    <origin xyz="0.09 0 0.1" rpy="0 1.5708 0"/>
+  </joint>
+  <link name="nose">
+    <visual>
+      <geometry>
+        <cylinder radius="0.015" length="0.03"/>
+      </geometry>
+      <material name="skin"/>
+    </visual>
+  </link>
+  <!-- Left Eye -->
+  <joint name="l_eye_yaw" type="revolute">
+    <parent link="head"/>
+    <child link="l_eye_yaw_link"/>
+    <origin xyz="0.08 0.04 0.13" rpy="0 0 0"/>
+    <axis xyz="0 0 1"/>
+    <limit lower="-0.5" upper="0.5" effort="5" velocity="5"/>
+  </joint>
+  <link name="l_eye_yaw_link"/>
+  <joint name="l_eye_pitch" type="revolute">
+    <parent link="l_eye_yaw_link"/>
+    <child link="l_eye"/>
+    <origin xyz="0 0 0" rpy="0 0 0"/>
+    <axis xyz="0 1 0"/>
+    <limit lower="-0.5" upper="0.5" effort="5" velocity="5"/>
+  </joint>
+  <link name="l_eye">
+    <visual>
+      <geometry>
+        <sphere radius="0.018"/>
+      </geometry>
+      <material name="white">
+        <color rgba="1.0 1.0 1.0 1.0"/>
+      </material>
+    </visual>
+    <!-- Pupil -->
+    <visual>
+      <origin xyz="0.015 0 0" rpy="0 0 0"/>
+      <geometry>
+        <sphere radius="0.006"/>
+      </geometry>
+      <material name="black">
+        <color rgba="0.0 0.0 0.0 1.0"/>
+      </material>
+    </visual>
+  </link>
+  <!-- Left Eyelids (Blinking) -->
+  <joint name="l_upper_lid_pitch" type="revolute">
+    <parent link="head"/>
+    <child link="l_upper_lid"/>
+    <origin xyz="0.08 0.04 0.13" rpy="0 0 0"/>
+    <axis xyz="0 1 0"/>
+    <limit lower="-0.6" upper="0.0" effort="5" velocity="10"/>
+  </joint>
+  <link name="l_upper_lid">
+    <visual>
+      <origin xyz="0.019 0 0.01" rpy="0 -0.5 0"/>
+      <geometry>
+        <box size="0.005 0.04 0.02"/>
+      </geometry>
+      <material name="skin"/>
+    </visual>
+  </link>
+  <joint name="l_lower_lid_pitch" type="revolute">
+    <parent link="head"/>
+    <child link="l_lower_lid"/>
+    <origin xyz="0.08 0.04 0.13" rpy="0 0 0"/>
+    <axis xyz="0 1 0"/>
+    <limit lower="0.0" upper="0.6" effort="5" velocity="10"/>
+  </joint>
+  <link name="l_lower_lid">
+    <visual>
+      <origin xyz="0.019 0 -0.01" rpy="0 0.5 0"/>
+      <geometry>
+        <box size="0.005 0.04 0.02"/>
+      </geometry>
+      <material name="skin"/>
+    </visual>
+  </link>
+  <!-- Right Eye -->
+  <joint name="r_eye_yaw" type="revolute">
+    <parent link="head"/>
+    <child link="r_eye_yaw_link"/>
+    <origin xyz="0.08 -0.04 0.13" rpy="0 0 0"/>
+    <axis xyz="0 0 1"/>
+    <limit lower="-0.5" upper="0.5" effort="5" velocity="5"/>
+  </joint>
+  <link name="r_eye_yaw_link"/>
+  <joint name="r_eye_pitch" type="revolute">
+    <parent link="r_eye_yaw_link"/>
+    <child link="r_eye"/>
+    <origin xyz="0 0 0" rpy="0 0 0"/>
+    <axis xyz="0 1 0"/>
+    <limit lower="-0.5" upper="0.5" effort="5" velocity="5"/>
+  </joint>
+  <link name="r_eye">
+    <visual>
+      <geometry>
+        <sphere radius="0.018"/>
+      </geometry>
+      <material name="white"/>
+    </visual>
+    <!-- Pupil -->
+    <visual>
+      <origin xyz="0.015 0 0" rpy="0 0 0"/>
+      <geometry>
+        <sphere radius="0.006"/>
+      </geometry>
+      <material name="black"/>
+    </visual>
+  </link>
+  <!-- Right Eyelids (Blinking) -->
+  <joint name="r_upper_lid_pitch" type="revolute">
+    <parent link="head"/>
+    <child link="r_upper_lid"/>
+    <origin xyz="0.08 -0.04 0.13" rpy="0 0 0"/>
+    <axis xyz="0 1 0"/>
+    <limit lower="-0.6" upper="0.0" effort="5" velocity="10"/>
+  </joint>
+  <link name="r_upper_lid">
+    <visual>
+      <origin xyz="0.019 0 0.01" rpy="0 -0.5 0"/>
+      <geometry>
+        <box size="0.005 0.04 0.02"/>
+      </geometry>
+      <material name="skin"/>
+    </visual>
+  </link>
+  <joint name="r_lower_lid_pitch" type="revolute">
+    <parent link="head"/>
+    <child link="r_lower_lid"/>
+    <origin xyz="0.08 -0.04 0.13" rpy="0 0 0"/>
+    <axis xyz="0 1 0"/>
+    <limit lower="0.0" upper="0.6" effort="5" velocity="10"/>
+  </joint>
+  <link name="r_lower_lid">
+    <visual>
+      <origin xyz="0.019 0 -0.01" rpy="0 0.5 0"/>
+      <geometry>
+        <box size="0.005 0.04 0.02"/>
+      </geometry>
+      <material name="skin"/>
+    </visual>
+  </link>
+  <!-- Upper Lip -->
+  <joint name="upper_lip_pitch" type="revolute">
+    <parent link="head"/>
+    <child link="upper_lip"/>
+    <origin xyz="0.09 0 0.07" rpy="0 0 0"/>
+    <axis xyz="0 1 0"/>
+    <limit lower="-0.2" upper="0.2" effort="5" velocity="5"/>
+  </joint>
+  <link name="upper_lip">
+    <visual>
+      <origin xyz="0.0 0 0" rpy="0 0 0"/>
+      <geometry>
+        <box size="0.01 0.06 0.015"/>
+      </geometry>
+      <material name="red">
+        <color rgba="0.8 0.3 0.3 1.0"/>
+      </material>
+    </visual>
+  </link>
+  <!-- Jaw and Lower Lip -->
   <joint name="jaw_pitch" type="revolute">
     <parent link="head"/>
     <child link="jaw"/>
-    <origin xyz="0 0.05 0.05" rpy="0 0 0"/>
-    <axis xyz="1 0 0"/>
-    <limit lower="-0.5" upper="0.0" effort="10" velocity="3"/>
+    <origin xyz="0.02 0 0.05" rpy="0 0 0"/>
+    <axis xyz="0 1 0"/>
+    <limit lower="-0.5" upper="0.0" effort="10" velocity="5"/>
   </joint>
   <link name="jaw">
     <visual>
-      <origin xyz="0 0.05 -0.05" rpy="0 0 0"/>
-      <geometry>
-        <box size="0.08 0.08 0.02"/>
-      </geometry>
-      <material name="skin"/>
+      <!-- Chin -->
+      <origin xyz="0.06 0 -0.03" rpy="0 0 0"/>
+      <geometry>
+        <box size="0.05 0.07 0.03"/>
+      </geometry>
+      <material name="skin"/>
+    </visual>
+    <visual>
+      <!-- Lower Lip -->
+      <origin xyz="0.07 0 0.0" rpy="0 0 0"/>
+      <geometry>
+        <box size="0.01 0.06 0.015"/>
+      </geometry>
+      <material name="red"/>
     </visual>
   </link>
